File: eda/SAO_Pin/SAO_Pin.kicad_pcb (KiCad board)
At the start: 2 copper layers, 0 parts

Commit message: basic 2032 cell power for SAO
Parts:
- added BT1: Battery_CR2032, 0_local:BatteryHolder_CR2032-BS-2-1_Front_backsilk, F.Cu at (131.3, 94.0)
- added JSAO1: Conn_02x03_SAO, 0_sao_v169bis:SAOv169-BADGEv2-PO-2x3, F.Cu at (143.4, 115.6)
Routing:
- net Net-(BT1-+): track 0.00 -> 25.9 mm
- net GND: track 0.00 -> 25.6 mm
Other:
- board outline added: 27.3 x 39.5 mm
