File: eda/SAO_Pin/SAO_Pin.kicad_sch (KiCad schematic)
At the start: 0 parts

Commit message: Initial template updates
Other:
- title: TEMPLATEPCB -> SAO_Pin
Changed lines of the file:
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@@
   (paper "USLetter")
   (title_block
-    (title "TEMPLATEPCB")
+    (title "SAO_Pin")
     (date "2025-02-09")
     (rev "1")

Commit message: basic 2032 cell power for SAO
Parts:
- added BT1: Battery_CR2032, 0_local:BatteryHolder_CR2032-BS-2-1_Front_backsilk, symbol Device:Battery_Cell
- added JSAO1: Conn_02x03_SAO, 0_sao_v169bis:SAOv169-BADGEv2-PO-2x3, symbol 0_local:Conn_02x03_SAO
Connections:
- new net: BT1.1 (+), JSAO1.1 (Pin_1)
- new net GND: BT1.2 (-), JSAO1.2 (Pin_2)
- no-connect marks 0 -> 4

Commit message: pcb updates
Parts:
- BT1: footprint 0_local:BatteryHolder_CR2032-BS-2-1_Front_backsilk -> 0_local:BatteryHolder_CR2032-BS-2-1_Back_backsilk
Changed lines of the file:
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@@
 			)
 		)
-		(property "Footprint" "0_local:BatteryHolder_CR2032-BS-2-1_Front_backsilk"
+		(property "Footprint" "0_local:BatteryHolder_CR2032-BS-2-1_Back_backsilk"
 			(at 137.16 139.446 90)
 			(effects
